Commit message: obstacle avoiding bot following Manhattan behaviour

File: task2/urdf/robot.urdf (robot description, URDF)
Before this commit: robot robot2, 8 links, 7 joints
Links:
- added link lidar_link, mass 0.1; collision cylinder length=0.04 radius=0.03; visual cylinder length=0.04 radius=0.03
Joints:
- added joint lidar_joint: type fixed, parent base_link, child lidar_link, origin xyz=-0.03 0 0.17 rpy=0 0 0
