Commit message: Task3

File: task3/urdf/maze.urdf (robot description, URDF)
Before this commit: robot my_maze, 1 links, 0 joints
Links:
- link maze_link: geometry collision mesh filename=file:///home/yash/ros2_ws/src/task3/meshes/maze_v1.stl scale=0.03 0.03 0.03; visual mesh filename=file:///home/yash/ros2_ws/src/task3/meshes/maze_v1.stl scale=0.03 0.03 0.03
